File: hardware/main-board/pcb/flip-segment-clock_main-board/flip-segment-clock_main-board.kicad_pcb (KiCad board)
At the start: 2 copper layers, 0 parts

Commit message: Refining design of the segment drivers
Parts:
- added BT1: CR2032, Battery:BatteryHolder_Keystone_1057_1x2032, F.Cu at (123.4, 63.9)
- added C1: 2.2 uF, Capacitor_SMD:C_0402_1005Metric, F.Cu at (117.4, 104.9)
- added C2: 22 uF, Capacitor_SMD:C_0402_1005Metric, F.Cu at (117.4, 106.8)
- added IC1: STM32G071CBT6, STM32G071CBT6:QFP50P900X900X160-48N, F.Cu at (145.0, 90.5)
- added IC2: DS3231MZ+TRL, SamacSys_Parts:SOIC127P600X175-8N, F.Cu at (110.0, 79.5)
- added IC3: TPS62177DQCR, SamacSys_Parts:SON50P200X300X80-11N, F.Cu at (113.9, 106.3)
- added J1: Barrel_Jack, Connector_BarrelJack:BarrelJack_SwitchcraftConxall_RAPC10U_Horizontal, F.Cu at (135.2, 94.3)
- added L1: 10 uH, Inductor_SMD:L_Coilcraft_LPS4018, F.Cu at (108.7, 106.6)
- added R1: 100k, Resistor_SMD:R_0402_1005Metric, F.Cu at (120.3, 104.9)
- added R2: 50k, Resistor_SMD:R_0402_1005Metric, F.Cu at (115.7, 77.2)
- added R3: 4.7k, Resistor_SMD:R_0402_1005Metric, F.Cu at (115.7, 79.2)
- added R4: 4.7k, Resistor_SMD:R_0402_1005Metric, F.Cu at (115.7, 81.2)
- added TP1: 32 kHz, TestPoint:TestPoint_Pad_D2.5mm, F.Cu at (119.4, 78.5)
Other:
- board outline added: 29.4 x 23 mm
